File: Hardware/RAMboard/RAMboard.kicad_pcb (KiCad board)
At the start: 2 copper layers, 21.6 x 38.1 mm, 4 parts, among them J1 RAMC_L, J2 RAMC_R, U1 FM18W08-SG

Commit message: Update capacitor value
Specify 100n as the decoupling capacitor value
Parts:
- C1: value C -> 100n
