File: Hardware/ROMboard/ROMboard.kicad_pcb (KiCad board)
At the start: 2 copper layers, 22.9 x 48.3 mm, 6 parts, among them J0 Conn_01x16, J1 Conn_01x16, J2 Conn_01x04, U1 M29F160

Commit message: Update capacitor value
Set decoupling capacitor value to 100n
Parts:
- C1: value C -> 100n
