File: Hardware/ROMboard/ROMboard.sch (KiCad schematic (older format))
At the start: 6 parts, among them J0 Conn_01x16, J1 Conn_01x16, J2 Conn_01x04, U1 M29F160

Commit message: Update capacitor value
Set decoupling capacitor value to 100n
Parts:
- C1: value C -> 100n
Changed lines of the file:
@@
 P 7300 1950
 F 0 "C1" V 7048 1950 50  0000 C CNN
-F 1 "C" V 7139 1950 50  0000 C CNN
+F 1 "100n" V 7139 1950 50  0000 C CNN
 F 2 "Capacitor_THT:CP_Radial_D5.0mm_P2.50mm" H 7338 1800 50  0001 C CNN
 F 3 "~" H 7300 1950 50  0001 C CNN
