File: Hardware/ROMStackable/ROMboard.kicad_pcb (KiCad board)
At the start: 2 copper layers, 22.9 x 54.6 mm, 10 parts, among them J0 Conn_01x16, J1 Conn_01x16, J2 Conn_01x04, U1 M29F160, U2 74LVC1G19

Commit message: Update capacitor values
Set decoupling capacitor values to 100n
Parts:
- C1, C2: value C -> 100n
