File: Hardware/Writeboi/progshield.kicad_pcb (KiCad board)
At the start: 2 copper layers, 121.9 x 81.3 mm, 14 parts, among them J1 GB-CART, J2 AUX_POW, SW1 SW_Push, U1 SST39SF040

Commit message: Update capacitor value
Set decoupling capacitor value to 100n
Parts:
- C1: value C -> 100n
