File: Hardware/ROMAdaptor/ROMAdaptor.kicad_pcb (KiCad board)
At the start: 2 copper layers, 29.2 x 43.2 mm, 4 parts, among them J1 Conn_01x16, J2 Conn_01x16, U1 SST39SF040

Commit message: Update capacitor value
Set decoupling capacitor value to 100n
Parts:
- C1: value C -> 100n
