File: Hardware/ROMAdaptor/ROMAdaptor.sch (KiCad schematic (older format))
At the start: 4 parts, among them J1 Conn_01x16, J2 Conn_01x16, U1 SST39SF040

Commit message: Update capacitor value
Set decoupling capacitor value to 100n
Parts:
- C1: value C -> 100n
Changed lines of the file:
@@
 P 3150 1050
 F 0 "C1" H 3265 1096 50  0000 L CNN
-F 1 "C" H 3265 1005 50  0000 L CNN
+F 1 "100n" H 3265 1005 50  0000 L CNN
 F 2 "Capacitor_THT:C_Disc_D3.8mm_W2.6mm_P2.50mm" H 3188 900 50  0001 C CNN
 F 3 "~" H 3150 1050 50  0001 C CNN
