File: Hardware/KiCad 6/Mainboard/Squareboi2.kicad_pcb (KiCad board)
At the start: 2 copper layers, 72 x 139 mm, 31 parts, among them J1 GB-CART, J10 TP_CLK, J11 TP_40, J12 TP_RST, J2 ROMC_L, J4 ROMC_C, J5 RAMC_L, J6 RAMC_R, J7 JTAG, J8 AUX_POW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

Commit message: Clean up Mainboard traces
Clean up disconnected traces
Routing:
- net /GBCLK: track 166.8 -> 163.6 mm
- net /A6: track 122.1 -> 119.0 mm
- net /A9: track 121.3 -> 118.3 mm
- net /D0: track 148.7 -> 147.5 mm
- net /A12: track 186.1 -> 185.2 mm
- net /A2: track 109.3 -> 108.5 mm
