File: Hardware/KiCad 6/ATF Devboard/ATF1502BR.kicad_pcb (KiCad board)
At the start: 2 copper layers, 60 x 80 mm, 31 parts, among them J1 USB_B, J2 Conn_01x02, J3 Conn_01x22, J4 Conn_02x05_Odd_Even, J5 Conn_01x22, J6 Conn_02x05_Odd_Even, SW1 SW_DIP_x06, SW4 SW_Push, SW5 SW_Push, U1 ATF1502-PLCC

Commit message: Clean up ATF Devboard traces
Clean up disconnected traces
Routing:
- net /LED0: track 6.50 -> 5.87 mm
Changed lines of the file:
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@@
   (segment (start 53.15863 33.97) (end 64.45 33.97) (width 0.25) (layer "F.Cu") (net 48))
   (segment (start 56.83 30.16) (end 56.83 31.43) (width 0.25) (layer "F.Cu") (net 49))
-  (segment (start 53.655 28.255) (end 53.02 28.255) (width 0.25) (layer "F.Cu") (net 49))
   (segment (start 53.02 28.255) (end 54.925 28.255) (width 0.25) (layer "F.Cu") (net 49))
   (segment (start 54.925 28.255) (end 56.83 30.16) (width 0.25) (layer "F.Cu") (net 49))
@@
   (zone (net 1) (net_name "GND") (layer "B.Cu") (hatch edge 0.508)
     (connect_pads (clearance 0.508))
-    (min_thickness 0.254)
+    (min_thickness 0.254) (filled_areas_thickness no)
     (fill yes (thermal_gap 0.508) (thermal_bridge_width 0.508) (smoothing fillet) (radius 2))
     (polygon
